File: esp_click_pcb/esp_click_pcb.kicad_sch (KiCad schematic)
At the start: 53 parts, among them J1 USB_C, SW1 BOOT, SW2 FLASH, SW3 BT1, SW4 BT2, SW5 BT3, SW6 BT4, U1 ESP32-C6-MINI, U2 HT7833, U4 BQ24075RGT

Commit message: pcb layout complete
Parts:
- D1, D2, D3: footprint LED_SMD:LED_0201_0603Metric -> LED_SMD:LED_0603_1608Metric
- TP2: value TestPoint -> GND
Changed lines of the file:
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@@
 			)
 		)
-		(property "Footprint" "LED_SMD:LED_0201_0603Metric"
+		(property "Footprint" "LED_SMD:LED_0603_1608Metric"
 			(at 154.94 87.63 0)
 			(effects
@@
 			)
 		)
-		(property "Footprint" "LED_SMD:LED_0201_0603Metric"
+		(property "Footprint" "LED_SMD:LED_0603_1608Metric"
 			(at 154.94 106.68 0)
 			(effects
@@
 			)
 		)
-		(property "Footprint" "LED_SMD:LED_0201_0603Metric"
+		(property "Footprint" "LED_SMD:LED_0603_1608Metric"
 			(at 154.94 96.52 0)
 			(effects
@@
 			)
 		)
-		(property "Value" "TestPoint"
+		(property "Value" "GND"
 			(at 40.64 187.9599 90)
 			(effects

Commit message: use rgb led directly
Parts:
- removed D1: R, LED_SMD:LED_0603_1608Metric, symbol Device:LED
- removed D2: G, LED_SMD:LED_0603_1608Metric, symbol Device:LED
- removed D3: B, LED_SMD:LED_0603_1608Metric, symbol Device:LED
- added LED1: RGB, XL-1615RGBC-RF:XL-1615RGBC-RF, symbol Device:LED_ARBG
- R12, R21: value 100R -> 33R
- R20: value 330R -> 100R
Connections:
- net +3.3V: now also LED1.1 (A)
- net at R20.1: now also LED1.2 (RK)
- net at R21.1: now also LED1.3 (BK)
- net at R12.1: now also LED1.4 (GK)
Other:
- moved on the sheet: R21

Commit message: update pcb design, rev2
Parts:
- removed R4: 10K, Resistor_SMD:R_0603_1608Metric, symbol Device:R
- R12, R21: value 33R -> 100R
Changed lines of the file:
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@@
 	(title_block
 		(title "ESP Click")
-		(date "2026-03-05")
-		(rev "1")
+		(date "2026-03-13")
+		(rev "2")
 		(company "Madhukar Temba")
 	)
@@
 			)
 		)
-		(property "Value" "33R"
+		(property "Value" "100R"
 			(at 146.05 101.6 90)
 			(effects
@@
 	)
 	(symbol
-		(lib_id "Device:R")
-		(at 147.32 68.58 180)
-		(unit 1)
-		(exclude_from_sim no)
-		(in_bom yes)
-		(on_board yes)
-		(dnp no)
-		(fields_autoplaced yes)
-		(property "Reference" "R4"
-			(at 149.86 67.3099 0)
-			(effects
-				(font
-					(size 1.27 1.27)
-				)
-				(justify right)
-			)
-		)
-		(property "Value" "10K"
-			(at 149.86 69.8499 0)
-			(effects
-				(font
-					(size 1.27 1.27)
-				)
-				(justify right)
-			)
-		)
-		(property "Footprint" "Resistor_SMD:R_0603_1608Metric"
-			(at 149.098 68.58 90)
-			(effects
-				(font
-					(size 1.27 1.27)
-				)
-				(hide yes)
-			)
-		)
-		(property "Datasheet" "~"
-			(at 147.32 68.58 0)
-			(effects
-				(font
-					(size 1.27 1.27)
-				)
-				(hide yes)
-			)
-		)
-		(property "Description" "Resistor"
-			(at 147.32 68.58 0)
-			(effects
-				(font
-					(size 1.27 1.27)
-				)
-				(hide yes)
-			)
-		)
-		(pin "1"
-		)
-		(pin "2"
-		)
-		(instances
-			(project "esp_click_pcb"
-				(path "/342a49d9-6002-45d3-9ef6-1f04f7424998"
-					(reference "R4")
-					(unit 1)
-				)
-			)
-		)
-	)
-	(symbol
 		(lib_id "Regulator_Linear:HT75xx-1-SOT89")
 		(at 215.9 129.54 0)
@@
 	)
 	(symbol
-		(lib_id "power:+3.3V")
-		(at 147.32 64.77 0)
-		(unit 1)
-		(exclude_from_sim no)
-		(in_bom yes)
-		(on_board yes)
-		(dnp no)
-		(fields_autoplaced yes)
-		(property "Reference" "#PWR09"
-			(at 147.32 68.58 0)
-			(effects
-				(font
-					(size 1.27 1.27)
-				)
-				(hide yes)
-			)
-		)
-		(property "Value" "+3.3V"
-			(at 147.32 59.69 0)
-			(effects
-				(font
-					(size 1.27 1.27)
-				)
-			)
-		)
-		(property "Footprint" ""
-			(at 147.32 64.77 0)
-			(effects
-				(font
-					(size 1.27 1.27)
-				)
-				(hide yes)
-			)
-		)
-		(property "Datasheet" ""
-			(at 147.32 64.77 0)
-			(effects
-				(font
-					(size 1.27 1.27)
-				)
-				(hide yes)
-			)
-		)
-		(property "Description" "Power symbol creates a global label with name \"+3.3V\""
-			(at 147.32 64.77 0)
-			(effects
-				(font
-					(size 1.27 1.27)
-				)
-				(hide yes)
-			)
-		)
-		(pin "1"
-		)
-		(instances
-			(project "esp_click_pcb"
-				(path "/342a49d9-6002-45d3-9ef6-1f04f7424998"
-					(reference "#PWR09")
-					(unit 1)
-				)
-			)
-		)
-	)
-	(symbol
 		(lib_id "Device:R")
 		(at 238.76 91.44 180)
@@
 			)
 		)
-		(property "Value" "33R"
+		(property "Value" "100R"
 			(at 146.05 92.71 90)
 			(effects

Commit message: rev 3
Parts:
- R9: value 1.5K -> 3K
Changed lines of the file:
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@@
 	(title_block
 		(title "ESP Click")
-		(date "2026-03-13")
-		(rev "2")
+		(date "2026-03-14")
+		(rev "3")
 		(company "Madhukar Temba")
 	)
@@
 			)
 		)
-		(property "Value" "1.5K"
+		(property "Value" "3K"
 			(at 109.22 184.1499 0)
 			(effects

Commit message: update cap value
Parts:
- C1: value 22uF -> 100uF
Changed lines of the file:
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@@
 	(title_block
 		(title "ESP Click")
-		(date "2026-03-14")
-		(rev "3")
+		(date "2026-03-19")
+		(rev "4")
 		(company "Madhukar Temba")
 	)
@@
 		(fields_autoplaced yes)
 		(property "Reference" "C1"
-			(at 218.44 134.62 90)
+			(at 229.87 133.3499 0)
 			(effects
 				(font
 					(size 1.27 1.27)
 				)
+				(justify left)
 			)
 		)
-		(property "Value" "22uF"
-			(at 220.98 134.62 90)
+		(property "Value" "100uF"
+			(at 229.87 135.8899 0)
 			(effects
 				(font
 					(size 1.27 1.27)
 				)
+				(justify left)
 			)
 		)
